File: Electro_biomed_proyecto.kicad_pcb (KiCad board)
At the start: 2 copper layers, 90 x 70 mm, 20 parts, among them J1 Conn_01x08_Socket, J2 Conn_01x04_Socket, J5 Conn_01x08_Socket, J7 Conn_01x04_Socket, SW1 SET, SW2 DOWN, SW3 UP, U3 AM2302

Commit message: Add files via upload
PCB que vamos a enviar a imprimir
Parts:
- added J3: MOSFET, Connector_PinSocket_2.54mm:PinSocket_1x03_P2.54mm_Vertical, F.Cu at (165.0, 78.0)
- added R7: R, Resistor_THT:R_Axial_DIN0204_L3.6mm_D1.6mm_P7.62mm_Horizontal, F.Cu at (159.0, 78.0)
- moved R6 34.4 mm to (163.0, 57.0), turned to 0 degrees
- moved R4 22.0 mm to (163.0, 71.0), turned to 0 degrees
- moved R5 8.22 mm to (163.0, 85.0), turned to 0 degrees
- moved SW2 6.18 mm to (177.5, 85.0)
- moved IN1 4.12 mm to (106.0, 96.5)
- moved OUT1 4.12 mm to (106.0, 52.0)
- moved U3 4.12 mm to (104.0, 81.5)
- moved IN2 4.07 mm to (178.0, 98.0)
- moved SW1 3.34 mm to (177.5, 71.0)
- moved SW3 1.46 mm to (177.5, 56.5)
Connections:
- IN2 pad 2: unconnected-(IN2-Pin_2-Pad2) -> /IO20
- J7 pad 2: unconnected-(J7-Pin_2-Pad2) -> /IO9
Routing:
- net /IO20: track 0.00 -> 65.1 mm, vias 0 -> 2
- net Net-(R5-Pad2): track 74.9 -> 25.9 mm, vias 0 -> 2
- net Net-(R6-Pad2): track 63.6 -> 19.7 mm, vias 2 -> 0
- net /GND: track 188.0 -> 153.4 mm
- net /IO9: track 0.00 -> 23.8 mm
- net /3V3: track 64.1 -> 85.8 mm, vias 0 -> 2
- net /IO7: track 31.3 -> 14.5 mm
- net Net-(R4-Pad2): track 41.3 -> 29.0 mm
- net /IO10: track 57.1 -> 49.1 mm
- net Net-(J3-Pin_1): track 0.00 -> 6.00 mm
- net /IO6: track 31.0 -> 26.9 mm
- net /IO3: track 48.0 -> 52.0 mm
- net /IO5: track 30.1 -> 26.8 mm
- net /12V: track 22.9 -> 20.2 mm
- net /GNDout: track 166.7 -> 164.6 mm
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