File: Electro_biomed_proyecto.kicad_sch (KiCad schematic)
At the start: 20 parts, among them J1 Conn_01x08_Socket, J2 Conn_01x04_Socket, J5 Conn_01x08_Socket, J7 Conn_01x04_Socket, SW1 SET, SW2 DOWN, SW3 UP, U3 AM2302

Commit message: Add files via upload
PCB que vamos a enviar a imprimir
Parts:
- added J3: MOSFET, Connector_PinSocket_2.54mm:PinSocket_1x03_P2.54mm_Vertical, symbol Connector:Conn_01x03_Socket
- added R7: R, Resistor_THT:R_Axial_DIN0204_L3.6mm_D1.6mm_P7.62mm_Horizontal, symbol Device:R
- J1, J5: footprint Connector_Harwin:Harwin_M20-89008xx_1x08_P2.54mm_Horizontal -> Connector_PinHeader_2.54mm:PinHeader_1x08_P2.54mm_Vertical
Connections:
- net 3V3: now also R7.2
- net GND: now also J3.3 (Pin_3)
- net IO20: now also IN2.2 (Pin_2), J3.2 (Pin_2)
- net IO9: now also J7.2 (Pin_2)
- new net: J3.1 (Pin_1), R7.1
